Commit message: new enviroment, ready to opti hyperparams on Kay

File: gym_environments/widowx_env/envs/URDFs/sphere.urdf (robot description, URDF)
Before this commit: robot myfirst, 1 links, 0 joints
Links:
- link base_link: mass None -> 0

File: gym_environments/widowx_env/envs/URDFs/widowx/widowx.urdf (robot description, URDF)
Before this commit: robot widowx, 10 links, 9 joints
Links:
- link gripper_aux_link: mass None -> 0
